File: kicad/photodiode_TIA/photodiode_TIA.kicad_sch (KiCad schematic)
At the start: 8 parts, among them J3 Conn_01x03_Pin, U1 MCP6001R

Commit message: added media
Other:
- title: (none) -> Precision Light Sensor AFE
Changed lines of the file:
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@@
 	(generator_version "9.0")
 	(paper "A4")
+	(title_block
+		(title "Precision Light Sensor AFE")
+		(date "2026-03-22")
+		(rev "v1.0")
+	)
 	(junction
 		(at 160.02 96.52)
